File: hardware/ArduTrxShield_CNC/kicad_source/ArduTrxShield.kicad_pcb (KiCad board)
At the start: 2 copper layers, 86.3 x 53 mm, 65 parts, among them CN1 60312202114509, CN2 ARDUINO, CN3 CON_KLINKE3, CN4 CON_KLINKE3, CN5 CONN_01X03, CN6 CONN_01X02, Q1 2N7002, Q2 2N7002, Q3 2N7002, SW1 TAST_HOR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

Commit message: update to version 1.1, changed C15 generated all data
Parts:
- C15: value 10u -> 470u; footprint capacitors:C_1206 -> capacitors:c_elec_8x10.5
- moved R23 5.60 mm to (124.0, 95.2)
- moved C15 2.61 mm to (124.1, 105.4)
- moved C12 1.78 mm to (121.0, 99.1), turned to 0 degrees
Connections:
- C15 pad 1: /SPKR -> Net-(C15-Pad1)
- C15 pad 2: Net-(C15-Pad2) -> /SPKR
- CN6 pad 1: Net-(C15-Pad2) -> Net-(C15-Pad1)
- R19 pad 1: Net-(C15-Pad2) -> Net-(C15-Pad1)
- U3 pad 5: Net-(C15-Pad2) -> Net-(C15-Pad1)
Routing:
- net GND: track 319.7 -> 287.4 mm
- net VCC: track 262.4 -> 236.9 mm
- net Net-(C15-Pad2): track 23.1 -> 0.00 mm
- net Net-(C15-Pad1): track 0.00 -> 17.2 mm
Other:
- board text added: "Copyright generationmake 2018 see full project documentation at http://ardutrx.generationmake.de This documentation describes Open Hardware and is licensed under the CERN OHL v. 1.2. You may redistribute and modify this documentation under the terms of the CERN OHL v.1.2. (http://ohwr.org/cernohl). This documentation is distributed WITHOUT ANY EXPRESS OR IMPLIED WARRANTY, INCLUDING OF MERCHANTABI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"
- board text added: "x1.1"
- board text removed: "x1.0"
