File: hardware/ArduTrxShield_CNC/kicad_source/ArduTrxShield.sch (KiCad schematic (older format))
At the start: 65 parts, among them CN1 60312202114509, CN2 ARDUINO, CN3 CON_KLINKE3, CN4 CON_KLINKE3, CN5 CONN_01X03, CN6 CONN_01X02, Q1 2N7002, Q2 2N7002, Q3 2N7002, SW1 TAST_HOR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

Commit message: update to version 1.1, changed C15 generated all data
Parts:
- removed C15: 10u, capacitors:C_1206, symbol C_1206
- added C15: 470u, capacitors:c_elec_8x10.5, symbol CP_Small
Other:
- note added: "Copyright generationmake 2018\nsee full project documentation at http://ardutrx.generationmake.de\n\nThis documentation describes Open Hardware and is licensed \nunder the CERN OHL v. 1.2.\nYou may redistribute and modify this documentation under the terms \nof the CERN OHL v.1.2. (http://ohwr.org/cernohl). This documentation \nis distributed WITHOUT ANY EXPRESS OR IMPLIED WARRANTY, \nINCLUDING O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"
Changed lines of the file:
@@
 Sheet 1 1
 Title "ArduTrx Shield CNC Version"
-Date "2018-06-11"
-Rev "x1.0"
+Date "2018-07-16"
+Rev "x1.1"
 Comp ""
 Comment1 ""
@@
 Text Notes 2950 7050 0    60   ~ 0
 LM4861 also works
-Text Notes 2050 1250 0    60   ~ 0
+Text Notes 700  3000 0    60   ~ 0
 filter for 2m version\nchebyshev low pass filter\ncutoff frequency: 185 MHz\npassband ripple: 0.5 dB\nimpedance: 50 Ohm
 $Comp
@@
 $EndComp
 Connection ~ 4350 5700
-$Comp
-L C_1206 C15
-U 1 1 5B0EACCD
-P 4350 5500
-F 0 "C15" H 4360 5570 50  0000 L CNN
-F 1 "10u" H 4360 5420 50  0000 L CNN
-F 2 "capacitors:C_1206" H 4350 5350 50  0001 C CNN
-F 3 "" H 4350 5500 50  0000 C CNN
-	1    4350 5500
-	1    0    0    -1
-$EndComp
 Wire Wire Line
 	4350 5600 4350 6350
@@
 Text Notes 2400 2650 0    60   ~ 0
 place R28..30 only if no filter necessary
+Text Notes 500  1250 0    47   ~ 0
+Copyright generationmake 2018\nsee full project documentation at http://ardutrx.generationmake.de\n\nThis   documentation   describes   Open   Hardware   and   is   licensed   \nunder   the CERN OHL v. 1.2.\nYou may redistribute and modify this documentation under the terms \nof the CERN OHL v.1.2. (http://ohwr.org/cernohl). This documentation \nis distributed WITHOUT   ANY   EXPRESS   OR   IMPLIED   WARRANTY, \nINCLUDING   OF MERCHANTABILITY,   SATISFACTORY   QUALITY   AND \nFITNESS   FOR   A PARTICULAR   PURPOSE.   Please   see   the   CERN   \nOHL   v.1.2  for   applicable conditions
+$Comp
+L CP_Small C15
+U 1 1 5B4C7944
+P 4350 5500
+F 0 "C15" H 4360 5570 50  0000 L CNN
+F 1 "470u" H 4360 5420 50  0000 L CNN
+F 2 "capacitors:c_elec_8x10.5" H 4350 5500 50  0001 C CNN
+F 3 "" H 4350 5500 50  0000 C CNN
+	1    4350 5500
+	-1   0    0    1
+$EndComp
 $EndSCHEMATC
