File: hardware/ArduTrxShield/kicad_source/ArduTrxShield.kicad_pcb (KiCad board)
At the start: 2 copper layers, 86.3 x 53 mm, 74 parts, among them CN1 60312202114509, CN2 ARDUINO, CN3 CON_KLINKE3, CN4 CON_KLINKE3, CN5 CONN_01X03, CN6 CONN_01X02, IC1 SN74LVC1T45, IC2 SN74LVC1T45, Q1 2N7002, Q2 2N7002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

Commit message: updated layout and schematic
Parts:
- added R32: DNI, resistors:R_0603, F.Cu at (119.3, 81.8)
- added S1: SW_DIP_x1, mechanical-switches:dip_1-300, F.Cu at (122.4, 83.0)
- moved C17 26.5 mm to (97.1, 90.2), turned to 90 degrees
- moved C18 25.7 mm to (97.1, 93.4), turned to 270 degrees
- moved IC1 25.4 mm to (99.9, 93.4)
- moved IC2 25.2 mm to (99.9, 90.2), turned to 180 degrees
- moved C20 24.3 mm to (102.6, 90.3), turned to 90 degrees
- moved C19 21.3 mm to (102.6, 93.4), turned to 270 degrees
- moved C14 18.6 mm to (97.0, 84.8)
- moved R27 17.0 mm to (124.5, 99.3), turned to 90 degrees
- moved C7 11.3 mm to (111.9, 123.2), turned to 270 degrees
- moved R4 11.3 mm to (99.9, 95.8), turned to 180 degrees
- moved R12 10.3 mm to (113.5, 85.7)
- moved C6 8.30 mm to (113.8, 122.8), turned to 270 degrees
- moved R5 7.86 mm to (100.0, 87.7), turned to 180 degrees
- moved R20 6.18 mm to (98.2, 98.5)
- moved C5 6.10 mm to (97.0, 83.2), turned to 180 degrees
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Connections:
- C6 pad 1: VAA -> VIN
- C7 pad 1: VAA -> VIN
- IC2 pad 3: /RXD -> /RXD_S
- R5 pad 1: /RXD -> /RXD_S
- U2 pad 3: VAA -> VIN
Routing:
- net VIO: track 53.5 -> 144.3 mm, vias 1 -> 3
- net /AF_OUT_R: track 90.4 -> 35.8 mm, vias 2 -> 1
- net GND: track 290.1 -> 239.8 mm, vias 2 -> 23
- net /RXD_S: track 0.00 -> 34.1 mm
- net VAA: track 23.0 -> 0.00 mm
- net VIN: track 4.45 -> 27.1 mm
- net /MIC_IN: track 47.6 -> 28.6 mm
- net /TXD: track 14.6 -> 27.1 mm
- net /SQ_R: track 21.4 -> 8.89 mm, vias 0 -> 1
- net VCC: track 225.4 -> 213.5 mm, vias 2 -> 5
- net /SQ: track 54.9 -> 66.8 mm, vias 0 -> 2
- net /ANT0: track 15.5 -> 24.6 mm
- net /ANT1: track 20.8 -> 29.2 mm
- net /RXD_R: track 42.9 -> 35.0 mm
- net /RXD: track 14.5 -> 6.61 mm
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- added copper zone on B.Cu, net GND
Other:
- board text added: "(c) 2018 generationmake"
- board text added: "Licensed under CERN OHL v.1.2"
- board text added: "x1.0"
- board text removed: "x1.1"

Commit message: generated gerber output
Routing:
- net GND: track 239.8 -> 248.2 mm, vias 23 -> 28
- net (no net): track 8.34 -> 0.00 mm, vias 5 -> 0
Other:
- board text added: "bot"
- board text added: "top"
Changed lines of the file:
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@@
     (area 54.624999 76.924999 141.075001 130.075001)
     (thickness 1.6)
-    (drawings 11)
-    (tracks 653)
+    (drawings 13)
+    (tracks 655)
     (zones 0)
     (modules 76)
@@
     (visible_elements FFFEFF7F)
     (pcbplotparams
-      (layerselection 0x00030_80000001)
-      (usegerberextensions false)
+      (layerselection 0x010e0_80000001)
+      (usegerberextensions true)
       (excludeedgelayer true)
       (linewidth 0.100000)
       (plotframeref false)
-      (viasonmask false)
+      (viasonmask true)
       (mode 1)
       (useauxorigin false)
@@
       (psa4output false)
       (plotreference true)
-      (plotvalue true)
+      (plotvalue false)
       (plotinvisibletext false)
       (padsonsilk false)
@@
     )
   )
+  (gr_text bot (at 138.9 113.3 90) (layer B.Cu)
+    (effects (font (size 1.5 1.5) (thickness 0.3)) (justify mirror))
+  )
+  (gr_text top (at 138.9 113.5 90) (layer F.Cu)
+    (effects (font (size 1.5 1.5) (thickness 0.3)))
+  )
   (gr_text "Licensed under CERN OHL v.1.2" (at 74.2 124.3) (layer F.SilkS)
     (effects (font (size 1.2 1.2) (thickness 0.3)))
@@
   (gr_line (start 141 130) (end 141 77) (angle 90) (layer Edge.Cuts) (width 0.15))
   (gr_line (start 54.7 130) (end 141 130) (angle 90) (layer Edge.Cuts) (width 0.15))
-  (segment (start 121.1 98.7) (end 121.1 97.3) (width 0.2) (layer B.Cu) (net 0))
-  (via (at 121.1 97.3) (size 0.8) (drill 0.4) (layers F.Cu B.Cu) (net 0))
-  (segment (start 98.9 100.1) (end 99.7 100.1) (width 0.2) (layer B.Cu) (net 0))
-  (via (at 99.9 100.3) (size 0.8) (drill 0.4) (layers F.Cu B.Cu) (net 0))
-  (segment (start 99.7 100.1) (end 99.9 100.3) (width 0.2) (layer B.Cu) (net 0))
-  (segment (start 115.7 96.1) (end 113.9 96.1) (width 0.2) (layer B.Cu) (net 0))
-  (via (at 113.9 96.1) (size 0.8) (drill 0.4) (layers F.Cu B.Cu) (net 0))
-  (segment (start 102.6 89.6) (end 103.2 89.6) (width 0.2) (layer B.Cu) (net 0))
-  (via (at 103.9 88.9) (size 0.8) (drill 0.4) (layers F.Cu B.Cu) (net 0))
-  (segment (start 103.2 89.6) (end 103.9 88.9) (width 0.2) (layer B.Cu) (net 0))
-  (segment (start 113.8 123.9) (end 113.8 124.1) (width 0.2) (layer B.Cu) (net 0))
-  (via (at 112.2 125.7) (size 0.8) (drill 0.4) (layers F.Cu B.Cu) (net 0))
-  (segment (start 113.8 124.1) (end 112.2 125.7) (width 0.2) (layer B.Cu) (net 0))
+  (via (at 113.95 96.15) (size 0.8) (drill 0.4) (layers F.Cu B.Cu) (net 1))
+  (segment (start 113.95 96.15) (end 113.9 96.1) (width 0.2) (layer F.Cu) (net 1))
+  (segment (start 115.6 96.15) (end 113.95 96.15) (width 0.2) (layer F.Cu) (net 1) (status 400000))
+  (segment (start 113.95 96.15) (end 113.9 96.1) (width 0.2) (layer B.Cu) (net 1))
+  (segment (start 121.1 98.65) (end 121.1 97.3) (width 0.2) (layer F.Cu) (net 1) (status 400000))
+  (via (at 121.1 97.3) (size 0.8) (drill 0.4) (layers F.Cu B.Cu) (net 1))
+  (segment (start 102.6 89.55) (end 103.25 89.55) (width 0.2) (layer F.Cu) (net 1) (status 400000))
+  (via (at 103.9 88.9) (size 0.8) (drill 0.4) (layers F.Cu B.Cu) (net 1))
+  (segment (start 103.25 89.55) (end 103.9 88.9) (width 0.2) (layer F.Cu) (net 1))
+  (segment (start 98.95 100.1) (end 99.8 100.1) (width 0.2) (layer F.Cu) (net 1) (status 400000))
+  (via (at 100 100.3) (size 0.8) (drill 0.4) (layers F.Cu B.Cu) (net 1))
+  (segment (start 99.8 100.1) (end 100 100.3) (width 0.2) (layer F.Cu) (net 1))
+  (segment (start 113.8 123.8) (end 113.8 124.1) (width 0.2) (layer F.Cu) (net 1) (status C00000))
+  (segment (start 113.8 124.1) (end 112.2 125.7) (width 0.2) (layer F.Cu) (net 1) (status 400000))
+  (via (at 112.2 125.7) (size 0.8) (drill 0.4) (layers F.Cu B.Cu) (net 1))
   (segment (start 57.25 105) (end 56.5 105) (width 0.2) (layer F.Cu) (net 1))
   (segment (start 56.5 105) (end 56.6 105.1) (width 0.2) (layer F.Cu) (net 1))

Commit message: generated and updated output data and pdfs
Parts:
- removed IC1, IC2: SN74LVC1T45, SOT_TO:SOT-23-6
- added U4: SN74LVC1T45, SOT_TO:SOT-23-6, F.Cu at (99.9, 93.4)
- added U5: SN74LVC1T45, SOT_TO:SOT-23-6, F.Cu at (99.9, 90.2)
- D1: value Led_Small -> Led_red
- D2: value Led_Small -> Led_yellow
- D3: value Led_Small -> Led_green
Changed lines of the file:
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@@
   (title_block
     (title "ArduTrx Shield")
-    (date 2018-07-18)
+    (date 2018-07-20)
     (rev x1.0)
   )
@@
       (effects (font (size 1 1) (thickness 0.15)))
     )
-    (fp_text value Led_Small (at 0 1.5) (layer F.Fab)
+    (fp_text value Led_red (at 0 1.5) (layer F.Fab)
       (effects (font (size 1 1) (thickness 0.15)))
     )
@@
       (effects (font (size 1 1) (thickness 0.15)))
     )
-    (fp_text value Led_Small (at 0 1.5) (layer F.Fab)
+    (fp_text value Led_yellow (at 0 1.5) (layer F.Fab)
       (effects (font (size 1 1) (thickness 0.15)))
     )
@@
       (effects (font (size 1 1) (thickness 0.15)))
     )
-    (fp_text value Led_Small (at 0 1.5) (layer F.Fab)
+    (fp_text value Led_green (at 0 1.5) (layer F.Fab)
       (effects (font (size 1 1) (thickness 0.15)))
     )
@@
     )
   )
-  (module SOT_TO:SOT-23-6 (layer F.Cu)
-    (at 99.9 93.4)
-    (descr "6-pin SOT-23 package")
-    (tags SOT-23-6)
-    (attr smd)
-    (fp_text reference IC1 (at 2.7 -5.5) (layer F.SilkS)
-      (effects (font (size 1 1) (thickness 0.15)))
-    )
-    (fp_text value SN74LVC1T45 (at 0 2.9) (layer F.Fab)
-      (effects (font (size 1 1) (thickness 0.15)))
-    )
-    (fp_circle (center -0.4 -1.7) (end -0.3 -1.7) (layer F.SilkS) (width 0.15))
-    (fp_line (start 0.25 -1.45) (end -0.25 -1.45) (layer F.SilkS) (width 0.15))
-    (fp_line (start 0.25 1.45) (end 0.25 -1.45) (layer F.SilkS) (width 0.15))
-    (fp_line (start -0.25 1.45) (end 0.25 1.45) (layer F.SilkS) (width 0.15))
-    (fp_line (start -0.25 -1.45) (end -0.25 1.45) (layer F.SilkS) (width 0.15))
-    (pad 1 smd rect (at -1.1 -0.95) (size 1.06 0.65) (layers F.Cu F.Paste F.Mask)
-      (net 3 VCC))
-    (pad 2 smd rect (at -1.1 0) (size 1.06 0.65) (layers F.Cu F.Paste F.Mask)
-      (net 1 GND))
-    (pad 3 smd rect (at -1.1 0.95) (size 1.06 0.65) (layers F.Cu F.Paste F.Mask)
-      (net 38 /TXD_R))
-    (pad 4 smd rect (at 1.1 0.95) (size 1.06 0.65) (layers F.Cu F.Paste F.Mask)
-      (net 25 /TXD))
-    (pad 6 smd rect (at 1.1 -0.95) (size 1.06 0.65) (layers F.Cu F.Paste F.Mask)
-      (net 67 VIO))
-    (pad 5 smd rect (at 1.1 0) (size 1.06 0.65) (layers F.Cu F.Paste F.Mask)
-      (net 1 GND))
-    (model TO_SOT_Packages_SMD.3dshapes/SOT-23-6.wrl
-      (at (xyz 0 0 0))
-      (scale (xyz 1 1 1))
-      (rotate (xyz 0 0 0))
-    )
-  )
-  (module SOT_TO:SOT-23-6 (layer F.Cu)
-    (at 99.9 90.2 180)
-    (descr "6-pin SOT-23 package")
-    (tags SOT-23-6)
-    (attr smd)
-    (fp_text reference IC2 (at -2.7 -5.9 180) (layer F.SilkS)
-      (effects (font (size 1 1) (thickness 0.15)))
-    )
-    (fp_text value SN74LVC1T45 (at 0 2.9 180) (layer F.Fab)
-      (effects (font (size 1 1) (thickness 0.15)))
-    )
-    (fp_circle (center -0.4 -1.7) (end -0.3 -1.7) (layer F.SilkS) (width 0.15))
-    (fp_line (start 0.25 -1.45) (end -0.25 -1.45) (layer F.SilkS) (width 0.15))
-    (fp_line (start 0.25 1.45) (end 0.25 -1.45) (layer F.SilkS) (width 0.15))
-    (fp_line (start -0.25 1.45) (end 0.25 1.45) (layer F.SilkS) (width 0.15))
-    (fp_line (start -0.25 -1.45) (end -0.25 1.45) (layer F.SilkS) (width 0.15))
-    (pad 1 smd rect (at -1.1 -0.95 180) (size 1.06 0.65) (layers F.Cu F.Paste F.Mask)
-      (net 67 VIO))
-    (pad 2 smd rect (at -1.1 0 180) (size 1.06 0.65) (layers F.Cu F.Paste F.Mask)
-      (net 1 GND))
-    (pad 3 smd rect (at -1.1 0.95 180) (size 1.06 0.65) (layers F.Cu F.Paste F.Mask)
-      (net 69 /RXD_S))
-    (pad 4 smd rect (at 1.1 0.95 180) (size 1.06 0.65) (layers F.Cu F.Paste F.Mask)
-      (net 39 /RXD_R))
-    (pad 6 smd rect (at 1.1 -0.95 180) (size 1.06 0.65) (layers F.Cu F.Paste F.Mask)
-      (net 3 VCC))
-    (pad 5 smd rect (at 1.1 0 180) (size 1.06 0.65) (layers F.Cu F.Paste F.Mask)
-      (net 1 GND))
-    (model TO_SOT_Packages_SMD.3dshapes/SOT-23-6.wrl
-      (at (xyz 0 0 0))
-      (scale (xyz 1 1 1))
-      (rotate (xyz 0 0 0))
-    )
-  )
   (module resistors:R_0603 (layer F.Cu)
     (at 135 82.5 180)
@@
     (tags DIP)
     (fp_text reference S1 (at -1 6.3) (layer F.SilkS)
-      (effects (font (size 1.4986 1.4986) (thickness 0.29972)))
-    )
-    (fp_text value SW_DIP_x1 (at 0 6.604) (layer F.SilkS)
+      (effects (font (size 1 1) (thickness 0.15)))
+    )
+    (fp_text value SW_DIP_x1 (at 0 6.604) (layer F.SilkS) hide
       (effects (font (size 1.524 1.4986) (thickness 0.29972)))
     )
@@
     )
   )
+  (module SOT_TO:SOT-23-6 (layer F.Cu)
+    (at 99.9 93.4)
+    (descr "6-pin SOT-23 package")
+    (tags SOT-23-6)
+    (attr smd)
+    (fp_text reference U4 (at 2.4 -5.2) (layer F.SilkS)
+      (effects (font (size 1 1) (thickness 0.15)))
+    )
+    (fp_text value SN74LVC1T45 (at 0 2.9) (layer F.Fab)
+      (effects (font (size 1 1) (thickness 0.15)))
+    )
+    (fp_circle (center -0.4 -1.7) (end -0.3 -1.7) (layer F.SilkS) (width 0.15))
+    (fp_line (start 0.25 -1.45) (end -0.25 -1.45) (layer F.SilkS) (width 0.15))
+    (fp_line (start 0.25 1.45) (end 0.25 -1.45) (layer F.SilkS) (width 0.15))
+    (fp_line (start -0.25 1.45) (end 0.25 1.45) (layer F.SilkS) (width 0.15))
+    (fp_line (start -0.25 -1.45) (end -0.25 1.45) (layer F.SilkS) (width 0.15))
+    (pad 1 smd rect (at -1.1 -0.95) (size 1.06 0.65) (layers F.Cu F.Paste F.Mask)
+      (net 3 VCC))
+    (pad 2 smd rect (at -1.1 0) (size 1.06 0.65) (layers F.Cu F.Paste F.Mask)
+      (net 1 GND))
+    (pad 3 smd rect (at -1.1 0.95) (size 1.06 0.65) (layers F.Cu F.Paste F.Mask)
+      (net 38 /TXD_R))
+    (pad 4 smd rect (at 1.1 0.95) (size 1.06 0.65) (layers F.Cu F.Paste F.Mask)
+      (net 25 /TXD))
+    (pad 6 smd rect (at 1.1 -0.95) (size 1.06 0.65) (layers F.Cu F.Paste F.Mask)
+      (net 67 VIO))
+    (pad 5 smd rect (at 1.1 0) (size 1.06 0.65) (layers F.Cu F.Paste F.Mask)
+      (net 1 GND))
+    (model TO_SOT_Packages_SMD.3dshapes/SOT-23-6.wrl
+      (at (xyz 0 0 0))
+      (scale (xyz 1 1 1))
+      (rotate (xyz 0 0 0))
+    )
+  )
+  (module SOT_TO:SOT-23-6 (layer F.Cu)
+    (at 99.9 90.2 180)
+    (descr "6-pin SOT-23 package")
+    (tags SOT-23-6)
+    (attr smd)
+    (fp_text reference U5 (at -2.2 -5.5 180) (layer F.SilkS)
+      (effects (font (size 1 1) (thickness 0.15)))
+    )
+    (fp_text value SN74LVC1T45 (at 0 2.9 180) (layer F.Fab)
+      (effects (font (size 1 1) (thickness 0.15)))
+    )
+    (fp_circle (center -0.4 -1.7) (end -0.3 -1.7) (layer F.SilkS) (width 0.15))
+    (fp_line (start 0.25 -1.45) (end -0.25 -1.45) (layer F.SilkS) (width 0.15))
+    (fp_line (start 0.25 1.45) (end 0.25 -1.45) (layer F.SilkS) (width 0.15))
+    (fp_line (start -0.25 1.45) (end 0.25 1.45) (layer F.SilkS) (width 0.15))
+    (fp_line (start -0.25 -1.45) (end -0.25 1.45) (layer F.SilkS) (width 0.15))
+    (pad 1 smd rect (at -1.1 -0.95 180) (size 1.06 0.65) (layers F.Cu F.Paste F.Mask)
+      (net 67 VIO))
+    (pad 2 smd rect (at -1.1 0 180) (size 1.06 0.65) (layers F.Cu F.Paste F.Mask)
+      (net 1 GND))
+    (pad 3 smd rect (at -1.1 0.95 180) (size 1.06 0.65) (layers F.Cu F.Paste F.Mask)
+      (net 69 /RXD_S))
+    (pad 4 smd rect (at 1.1 0.95 180) (size 1.06 0.65) (layers F.Cu F.Paste F.Mask)
+      (net 39 /RXD_R))
+    (pad 6 smd rect (at 1.1 -0.95 180) (size 1.06 0.65) (layers F.Cu F.Paste F.Mask)
+      (net 3 VCC))
+    (pad 5 smd rect (at 1.1 0 180) (size 1.06 0.65) (layers F.Cu F.Paste F.Mask)
+      (net 1 GND))
+    (model TO_SOT_Packages_SMD.3dshapes/SOT-23-6.wrl
+      (at (xyz 0 0 0))
+      (scale (xyz 1 1 1))
+      (rotate (xyz 0 0 0))
+    )
+  )
   (gr_text bot (at 138.9 113.3 90) (layer B.Cu)
     (effects (font (size 1.5 1.5) (thickness 0.3)) (justify mirror))
@@
   (via (at 113.95 96.15) (size 0.8) (drill 0.4) (layers F.Cu B.Cu) (net 1))
   (segment (start 113.95 96.15) (end 113.9 96.1) (width 0.2) (layer F.Cu) (net 1))
-  (segment (start 115.6 96.15) (end 113.95 96.15) (width 0.2) (layer F.Cu) (net 1) (status 400000))
+  (segment (start 115.6 96.15) (end 113.95 96.15) (width 0.2) (layer F.Cu) (net 1))
   (segment (start 113.95 96.15) (end 113.9 96.1) (width 0.2) (layer B.Cu) (net 1))
-  (segment (start 121.1 98.65) (end 121.1 97.3) (width 0.2) (layer F.Cu) (net 1) (status 400000))
+  (segment (start 121.1 98.65) (end 121.1 97.3) (width 0.2) (layer F.Cu) (net 1))
   (via (at 121.1 97.3) (size 0.8) (drill 0.4) (layers F.Cu B.Cu) (net 1))
-  (segment (start 102.6 89.55) (end 103.25 89.55) (width 0.2) (layer F.Cu) (net 1) (status 400000))
+  (segment (start 102.6 89.55) (end 103.25 89.55) (width 0.2) (layer F.Cu) (net 1))
   (via (at 103.9 88.9) (size 0.8) (drill 0.4) (layers F.Cu B.Cu) (net 1))
   (segment (start 103.25 89.55) (end 103.9 88.9) (width 0.2) (layer F.Cu) (net 1))
-  (segment (start 98.95 100.1) (end 99.8 100.1) (width 0.2) (layer F.Cu) (net 1) (status 400000))
+  (segment (start 98.95 100.1) (end 99.8 100.1) (width 0.2) (layer F.Cu) (net 1))
   (via (at 100 100.3) (size 0.8) (drill 0.4) (layers F.Cu B.Cu) (net 1))
   (segment (start 99.8 100.1) (end 100 100.3) (width 0.2) (layer F.Cu) (net 1))
-  (segment (start 113.8 123.8) (end 113.8 124.1) (width 0.2) (layer F.Cu) (net 1) (status C00000))
-  (segment (start 113.8 124.1) (end 112.2 125.7) (width 0.2) (layer F.Cu) (net 1) (status 400000))
+  (segment (start 113.8 123.8) (end 113.8 124.1) (width 0.2) (layer F.Cu) (net 1))
+  (segment (start 113.8 124.1) (end 112.2 125.7) (width 0.2) (layer F.Cu) (net 1))
   (via (at 112.2 125.7) (size 0.8) (drill 0.4) (layers F.Cu B.Cu) (net 1))
   (segment (start 57.25 105) (end 56.5 105) (width 0.2) (layer F.Cu) (net 1))

Commit message: updated schematic and layout of ArduTrxShield to version 1.1, see CHANGES.txt for details
Parts:
- added CN7: 691322310002, CON_wuerth:WR-TBL_691322310002, F.Cu at (61.6, 122.1)
- added R33: 4k7, resistors:R_0603, F.Cu at (98.0, 110.0)
- added R34: 4k7, resistors:R_0603, F.Cu at (98.0, 104.8)
- added R35: 100k, resistors:R_0603, F.Cu at (71.2, 123.1)
- added R36: 20k, resistors:R_0603, F.Cu at (67.5, 123.1)
- CN3: footprint CON_lumberg:1503_08 -> CON_lumberg:1503_07
- R12: value 100 -> 4k7
- R16, R31: value 100 -> 1k
- R17: value 330 -> 300
- R2, R21: value 1k -> 4k7
- moved R18 14.3 mm to (60.9, 118.8), turned to 180 degrees
- moved CN5 13.4 mm to (56.7, 114.0), turned to 0 degrees
- moved R2 3.00 mm to (98.0, 115.2), turned to 90 degrees
- moved D2 2.34 mm to (137.0, 87.8)
- moved D3 2.34 mm to (137.0, 80.8)
- moved D1 2.27 mm to (137.0, 84.2)
- moved SW2 0.60 mm to (131.0, 121.8)
- moved CN4 0.54 mm to (141.5, 106.8)
- moved CN3 0.50 mm to (141.5, 95.0)
Connections:
- CN2 pad 10: /KEYPAD_10 -> (no net)
- CN2 pad 15: Net-(CN2-Pad15) -> (no net)
- CN2 pad 16: Net-(CN2-Pad16) -> (no net)
- CN2 pad 17: Net-(CN2-Pad17) -> (no net)
- CN2 pad 23: /KEYPAD_A0 -> (no net)
- CN2 pad 28: Net-(CN2-Pad28) -> (no net)
- CN2 pad 29: Net-(CN2-Pad29) -> (no net)
- CN2 pad 31: Net-(CN2-Pad31) -> (no net)
- CN2 pad 4: /KEYPAD_4 -> (no net)
- CN2 pad 5: /KEYPAD_5 -> (no net)
- CN2 pad 6: /KEYPAD_6 -> (no net)
- CN2 pad 7: /KEYPAD_7 -> (no net)
- CN2 pad 8: /KEYPAD_8 -> (no net)
- CN2 pad 9: /KEYPAD_9 -> (no net)
- R2 pad 1: VCC -> Net-(Q1-Pad1)
- R2 pad 2: /H_L -> GND
- U1 pad 11: Net-(U1-Pad11) -> (no net)
- U1 pad 13: Net-(U1-Pad13) -> (no net)
- U1 pad 14: Net-(U1-Pad14) -> (no net)
- U1 pad 15: Net-(U1-Pad15) -> (no net)
- U1 pad 2: Net-(U1-Pad2) -> (no net)
- U1 pad 4: Net-(U1-Pad4) -> (no net)
Routing:
- net VIN: track 27.1 -> 74.5 mm
- net /GPS_RX: track 36.9 -> 55.0 mm, vias 1 -> 2
- net VCC: track 213.5 -> 198.2 mm
- net GND: track 248.2 -> 237.9 mm, vias 28 -> 27
- net Net-(CN5-Pad3): track 11.1 -> 3.55 mm
- net Net-(CN3-Pad3): track 0.00 -> 6.60 mm
- net +5V: track 35.8 -> 40.5 mm
- net /SPKR: track 5.31 -> 8.69 mm
- net Net-(Q3-Pad1): track 1.27 -> 2.82 mm
- net Net-(Q2-Pad1): track 1.27 -> 2.82 mm
- net Net-(Q1-Pad1): track 1.72 -> 3.27 mm
- net /H_L: track 7.23 -> 5.87 mm
- net /AF_OUT_R: track 35.8 -> 37.1 mm
- net /PD_Q: track 42.7 -> 41.7 mm
- net /PTT_Q: track 34.9 -> 35.6 mm
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Other:
- board size 86.3 x 53 mm -> 84.8 x 53 mm
- board text added: "1.1"
- board text removed: "x1.0"
