File: hardware/ArduTrxShield/kicad_source/ArduTrxShield.sch (KiCad schematic (older format))
At the start: 74 parts, among them CN1 60312202114509, CN2 ARDUINO, CN3 CON_KLINKE3, CN4 CON_KLINKE3, CN5 CONN_01X03, CN6 CONN_01X02, IC1 SN74LVC1T45, IC2 SN74LVC1T45, Q1 2N7002, Q2 2N7002, Q3 2N7002, SW1 TAST_HOR, SW2 ALPS_EC11E, U1 DRA818, U2 LT1085, U3 LM4871

Commit message: updated layout and schematic
Parts:
- added R32: DNI, resistors:R_0603, symbol R_1206
- added S1: SW_DIP_x1, mechanical-switches:dip_1-300, symbol SW_DIP_x1
Connections:
- net labels added: RXD_S
- net labels removed: VAA
- wire segments 237 -> 244

Commit message: generated and updated output data and pdfs
Parts:
- D1: value Led_Small -> Led_red
- D2: value Led_Small -> Led_yellow
- D3: value Led_Small -> Led_green
- renumbered IC1 to U4, IC2 to U5
Connections:
- wire segments 244 -> 247
Other:
- moved on the sheet: CN5, D1, D2, R1, R16, R18, R31, R32, R6, S1

Commit message: updated schematic and layout of ArduTrxShield to version 1.1, see CHANGES.txt for details
Parts:
- added CN7: 691322310002, CON_wuerth:WR-TBL_691322310002, symbol CON_wuerth:691322310002
- added R33, R34: 4k7, resistors:R_0603, symbol R_1206
- added R35: 100k, resistors:R_0603, symbol R_1206
- added R36: 20k, resistors:R_0603, symbol R_1206
- CN3: footprint CON_lumberg:1503_08 -> CON_lumberg:1503_07
- R12: value 100 -> 4k7
- R16, R31: value 100 -> 1k
- R17: value 330 -> 300
- R2, R21: value 1k -> 4k7
Connections:
- wire segments 247 -> 321

Commit message: fixed schematic symbol links to library
Parts:
- C1, C10, C11, C12, C13, C14, C16, C17, C18, C19, C2, C20, C3, C4, C5, C6, C7, C8, C9: symbol C_1206 -> devices:C_0603
- C15: symbol CP_Small -> devices:CP_Small
- CN1: symbol 60312202114509 -> CON_wuerth:60312202114509
- CN2: symbol ARDUINO -> MODULE_compute:ARDUINO
- CN3, CN4: symbol CON_KLINKE3 -> mechanical-connectors:CON_KLINKE3
- CN5: symbol CONN_01X03 -> mechanical-connectors:CONN_01X03
- CN6: symbol CONN_01X02 -> mechanical-connectors:CONN_01X02
- D1, D2, D3: symbol Led_Small -> devices:Led_Small
- D4: symbol D_Schottky_Small -> devices:D_Schottky_Small
- L1, L2, L3: symbol 744912156 -> L_filter:744912156
- Q1, Q2, Q3: symbol Q_NMOS_GSD -> devices:Q_NMOS_GSD
- R1, R10, R11, R12, R13, R14, R15, R16, R17, R18, R19, R2, R20, R21, R22, R23, R24, R25, R26, R27, R28, R29, R3, R30, R31, R32, R33, R34, R35, R36, R4, R5, R6, R7, R8, R9: symbol R_1206 -> devices:R_0603
- S1: symbol SW_DIP_x1 -> mechanical-switches:SW_DIP_x1
- SW1: symbol TAST_HOR -> mechanical-switches:TAST_HOR
- SW2: symbol ALPS_EC11E -> mechanical-switches:ALPS_EC11E
- U1: symbol DRA818 -> MODULE_RF:DRA818
- U2: symbol LT1085 -> voltage-regulators:LT1085
- U3: symbol LM4871 -> IC_audio:LM4871
- U4, U5: symbol SN74LVC1T45 -> IC_levelshifter:SN74LVC1T45
