File: hardware/ArduTrxDMRShield/kicad_source/ArduTrxDMRShield.sch (KiCad schematic (older format))
At the start: 78 parts, among them CN1 60312202114509, CN2 ARDUINO, CN3 CON_KLINKE3, CN4 CON_KLINKE3, CN5 CONN_01X03, CN6 CONN_01X02, CN7 691322310002, Q2 2N7002, Q3 2N7002, SW1 TAST_HOR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

Commit message: corrected schematic, updated layout
Parts:
- removed D4: BAT46ZFILM, diodes:SOD-123, symbol devices:D_Schottky_Small
- removed L1, L2: 744912156, L_filter:WE-CAIR_4248, symbol L_filter:744912156
- removed R21: 4k7, resistors:R_0603, symbol devices:R_0603
- removed R22: 100, resistors:R_0603, symbol devices:R_0603
- removed R28, R29: DNI, resistors:R_0603, symbol devices:R_0603
- added Q1, Q4: 2N7002, SOT_TO:SOT-23, symbol devices:Q_NMOS_GSD
- added R2, R3: 100, resistors:R_0603, symbol devices:R_0603
- C1: value 30p -> 10u; footprint capacitors:C_0603 -> capacitors:C_0805
- C2: value 47p -> 100n
Connections:
- net labels added: PD_Q_1, PD_Q_2, PTT_Q_1, PTT_Q_2, SQ_Q
- net labels removed: ANT1, ANT2, KEYPAD_6, KEYPAD_7
- wire segments 314 -> 316
- no-connect marks 20 -> 18
Other:
- moved on the sheet: D3, R11, R12, R7, R9

Commit message: updated schematic and layout, connected some nets to 3.3v output of DMR818
Parts:
- added R21: 4k7, resistors:R_0603, symbol devices:R_0603
Connections:
- net labels added: +3V3, TRANSMIT
- wire segments 316 -> 323
- no-connect marks 18 -> 16
Other:
- note added: "set VCC to 5.0 V\n(max. supply voltage of DMR818)"
- note removed: "set VCC to 4.5 V\n(max. supply voltage of DRA818)"
- moved on the sheet: D1, D2, D3, Q4, R7
Changed lines of the file:
@@
 Text Label 9250 3200 0    60   ~ 0
 SQ_R
-Text Label 7350 750  0    60   ~ 0
+Text Label 8250 750  0    60   ~ 0
 SQ
 $Comp
 L devices:Led_Small D3
 U 1 1 5B0B32C3
-P 7900 750
-F 0 "D3" H 7850 875 50  0000 L CNN
-F 1 "Led_green" H 7725 650 50  0000 L CNN
-F 2 "LEDs:LED_0603" V 7900 750 50  0001 C CNN
-F 3 "" V 7900 750 50  0000 C CNN
-	1    7900 750
-	1    0    0    -1
+P 7550 1200
+F 0 "D3" H 7500 1325 50  0000 L CNN
+F 1 "Led_green" H 7375 1100 50  0000 L CNN
+F 2 "LEDs:LED_0603" V 7550 1200 50  0001 C CNN
+F 3 "" V 7550 1200 50  0000 C CNN
+	1    7550 1200
+	-1   0    0    1
 $EndComp
 $Comp
 L devices:R_0603 R7
 U 1 1 5B0B331A
-P 7600 750
-F 0 "R7" H 7630 770 50  0000 L CNN
-F 1 "1k" H 7630 710 50  0000 L CNN
-F 2 "resistors:R_0603" H 7600 600 50  0001 C CNN
-F 3 "" H 7600 750 50  0000 C CNN
-	1    7600 750
+P 7200 1200
+F 0 "R7" H 7230 1220 50  0000 L CNN
+F 1 "1k" H 7230 1160 50  0000 L CNN
+F 2 "resistors:R_0603" H 7200 1050 50  0001 C CNN
+F 3 "" H 7200 1200 50  0000 C CNN
+	1    7200 1200
 	0    1    1    0
-$EndComp
-$Comp
-L power-supply:VCC #PWR01
-U 1 1 5B0B338E
-P 8100 700
-F 0 "#PWR01" H 8100 550 50  0001 C CNN
-F 1 "VCC" H 8100 850 50  0000 C CNN
-F 2 "" H 8100 700 50  0000 C CNN
-F 3 "" H 8100 700 50  0000 C CNN
-	1    8100 700
-	1    0    0    -1
 $EndComp
 NoConn ~ 4550 1700
@@
 	0    1    1    0
 $EndComp
-$Comp
-L power-supply:VCC #PWR014
-U 1 1 5B0B5B5B
-P 8300 2250
-F 0 "#PWR014" H 8300 2100 50  0001 C CNN
-F 1 "VCC" H 8300 2400 50  0000 C CNN
-F 2 "" H 8300 2250 50  0000 C CNN
-F 3 "" H 8300 2250 50  0000 C CNN
-	1    8300 2250
-	0    1    1    0
-$EndComp
 Text Label 5400 3450 0    60   ~ 0
 MIC_IN
@@
 F 3 "" V 10500 1200 50  0000 C CNN
 	1    10500 1200
-	1    0    0    -1
+	-1   0    0    1
 $EndComp
 $Comp
@@
 F 3 "" V 10500 800 50  0000 C CNN
 	1    10500 800
-	1    0    0    -1
+	-1   0    0    1
 $EndComp
 $Comp
 L power-supply:GND #PWR015
 U 1 1 5B0B6605
-P 9850 1300
-F 0 "#PWR015" H 9850 1050 50  0001 C CNN
-F 1 "GND" H 9850 1150 50  0000 C CNN
-F 2 "" H 9850 1300 50  0000 C CNN
-F 3 "" H 9850 1300 50  0000 C CNN
-	1    9850 1300
-	1    0    0    -1
-$EndComp
-$Comp
-L power-supply:VCC #PWR016
-U 1 1 5B0B665E
-P 10700 700
-F 0 "#PWR016" H 10700 550 50  0001 C CNN
-F 1 "VCC" H 10700 850 50  0000 C CNN
-F 2 "" H 10700 700 50  0000 C CNN
-F 3 "" H 10700 700 50  0000 C CNN
-	1    10700 700
+P 10700 1250
+F 0 "#PWR015" H 10700 1000 50  0001 C CNN
+F 1 "GND" H 10700 1100 50  0000 C CNN
+F 2 "" H 10700 1250 50  0000 C CNN
+F 3 "" H 10700 1250 50  0000 C CNN
+	1    10700 1250
 	1    0    0    -1
 $EndComp
 Text Label 9400 800  0    60   ~ 0
-PTT
+TRANSMIT
 $Comp
 L power-supply:GND #PWR017
@@
 	9900 3200 6450 3200
 Wire Wire Line
-	8000 750  8100 750
-Wire Wire Line
-	8100 750  8100 700
-Wire Wire Line
-	7800 750  7700 750
-Wire Wire Line
 	6350 1600 5750 1600
 Wire Wire Line
@@
 Connection ~ 7900 1500
 Wire Wire Line
-	10700 700  10700 800
-Wire Wire Line
 	10700 1200 10600 1200
 Wire Wire Line
 	10050 1200 9850 1200
 Wire Wire Line
-	9850 1200 9850 1300
-Wire Wire Line
 	10250 1200 10400 1200
 Wire Wire Line
@@
 Wire Wire Line
 	10600 800  10700 800
-Connection ~ 10700 800
 Wire Wire Line
 	3650 1700 3650 2000
@@
 Wire Wire Line
 	600  6500 1350 6500
-Text Label 2100 7100 0    60   ~ 0
+Text Label 1800 7250 0    60   ~ 0
 SQ
 Text Label 750  6500 0    60   ~ 0
@@
 	0    1    1    0
 $EndComp
-$Comp
-L power-supply:VCC #PWR037
-U 1 1 5B0EC4F1
-P 3450 5150
-F 0 "#PWR037" H 3450 5000 50  0001 C CNN
-F 1 "VCC" H 3450 5300 50  0000 C CNN
-F 2 "" H 3450 5150 50  0000 C CNN
-F 3 "" H 3450 5150 50  0000 C CNN
-	1    3450 5150
-	1    0    0    -1
-$EndComp
 Wire Wire Line
 	2350 5450 3150 5450
@@
 MIC_IN
 Text Notes 2900 3350 0    60   ~ 0
-set VCC to 4.5 V\n(max. supply voltage of DRA818)
+set VCC to 5.0 V\n(max. supply voltage of DMR818)
 $Comp
 L mechanical-connectors:CON_KLINKE3 CN4
@@
 	6700 4550 7250 4550
 Connection ~ 6700 4350
-$Comp
-L power-supply:VCC #PWR047
-U 1 1 5B4D63EC
-P 6600 3400
-F 0 "#PWR047" H 6600 3250 50  0001 C CNN
-F 1 "VCC" H 6600 3550 50  0000 C CNN
-F 2 "" H 6600 3400 50  0000 C CNN
-F 3 "" H 6600 3400 50  0000 C CNN
-	1    6600 3400
-	1    0    0    -1
-$EndComp
 Wire Wire Line
 	7000 4150 6600 4150
@@
 F 3 "" H 5400 4550 50  0000 C CNN
 	1    5400 4550
-	1    0    0    -1
-$EndComp
-$Comp
-L power-supply:VCC #PWR052
-U 1 1 5B4D76BB
-P 5400 4250
-F 0 "#PWR052" H 5400 4100 50  0001 C CNN
-F 1 "VCC" H 5400 4400 50  0000 C CNN
-F 2 "" H 5400 4250 50  0000 C CNN
-F 3 "" H 5400 4250 50  0000 C CNN
-	1    5400 4250
-	1    0    0    -1
-$EndComp
-$Comp
-L power-supply:VCC #PWR053
-U 1 1 5B4D779E
-P 5700 4250
-F 0 "#PWR053" H 5700 4100 50  0001 C CNN
-F 1 "VCC" H 5700 4400 50  0000 C CNN
-F 2 "" H 5700 4250 50  0000 C CNN
-F 3 "" H 5700 4250 50  0000 C CNN
-	1    5700 4250
 	1    0    0    -1
 $EndComp
@@
 Wire Wire Line
 	5100 2700 5100 2600
-NoConn ~ 5750 1500
-NoConn ~ 5750 1700
 $Comp
 L power-supply:GND #PWR0101
@@
 	5650 2800 5650 2850
 $Comp
-L devices:Q_NMOS_GSD Q4
-U 1 1 5BD5563D
-P 7150 950
-F 0 "Q4" H 7450 1000 50  0000 R CNN
-F 1 "2N7002" H 7800 900 50  0000 R CNN
-F 2 "SOT_TO:SOT-23" H 7350 1050 50  0001 C CNN
-F 3 "" H 7150 950 50  0000 C CNN
-	1    7150 950
-	1    0    0    -1
-$EndComp
-$Comp
 L power-supply:GND #PWR019
 U 1 1 5BD8AD71
-P 7250 1200
-F 0 "#PWR019" H 7250 950 50  0001 C CNN
-F 1 "GND" H 7250 1050 50  0000 C CNN
-F 2 "" H 7250 1200 50  0000 C CNN
-F 3 "" H 7250 1200 50  0000 C CNN
-	1    7250 1200
-	1    0    0    -1
-$EndComp
-Wire Wire Line
-	7250 1150 7250 1200
-Wire Wire Line
-	7500 750  7250 750
+P 8150 1200
+F 0 "#PWR019" H 8150 950 50  0001 C CNN
+F 1 "GND" H 8150 1050 50  0000 C CNN
+F 2 "" H 8150 1200 50  0000 C CNN
+F 3 "" H 8150 1200 50  0000 C CNN
+	1    8150 1200
+	1    0    0    -1
+$EndComp
 Wire Wire Line
 	6200 1400 6200 950
-Wire Wire Line
-	6200 950  6950 950
 Wire Wire Line
 	5750 1400 6200 1400
@@
 Text Label 5850 1400 0    60   ~ 0
 SQ_Q
-Wire Wire Line
-	1750 7100 2400 7100
+$Comp
+L power-supply:+3V3 #PWR064
+U 1 1 5BFE47D9
+P 9850 1150
+F 0 "#PWR064" H 9850 1000 50  0001 C CNN
+F 1 "+3V3" H 9865 1323 50  0000 C CNN
+F 2 "" H 9850 1150 50  0000 C CNN
+F 3 "" H 9850 1150 50  0000 C CNN
+	1    9850 1150
+	1    0    0    -1
+$EndComp
+$Comp
+L power-supply:+3V3 #PWR037
+U 1 1 5BFE4BFE
+P 6500 1700
+F 0 "#PWR037" H 6500 1550 50  0001 C CNN
+F 1 "+3V3" H 6515 1873 50  0000 C CNN
+F 2 "" H 6500 1700 50  0000 C CNN
+F 3 "" H 6500 1700 50  0000 C CNN
+	1    6500 1700
+	1    0    0    -1
+$EndComp
+Wire Wire Line
+	5750 1700 6500 1700
+$Comp
+L devices:Q_NMOS_GSD Q4
+U 1 1 5BD5563D
+P 8050 950
+F 0 "Q4" H 8350 1000 50  0000 R CNN
+F 1 "2N7002" H 8700 900 50  0000 R CNN
+F 2 "SOT_TO:SOT-23" H 8250 1050 50  0001 C CNN
+F 3 "" H 8050 950 50  0000 C CNN
+	1    8050 950
+	1    0    0    -1
+$EndComp
+$Comp
+L power-supply:+3V3 #PWR053
+U 1 1 5C001438
+P 8300 2250
+F 0 "#PWR053" H 8300 2100 50  0001 C CNN
+F 1 "+3V3" V 8315 2378 50  0000 L CNN
+F 2 "" H 8300 2250 50  0000 C CNN
+F 3 "" H 8300 2250 50  0000 C CNN
+	1    8300 2250
+	0    1    1    0
+$EndComp
+$Comp
+L power-supply:+3V3 #PWR016
+U 1 1 5C001CC5
+P 5400 4250
+F 0 "#PWR016" H 5400 4100 50  0001 C CNN
+F 1 "+3V3" H 5415 4423 50  0000 C CNN
+F 2 "" H 5400 4250 50  0000 C CNN
+F 3 "" H 5400 4250 50  0000 C CNN
+	1    5400 4250
+	1    0    0    -1
+$EndComp
+$Comp
+L power-supply:+3V3 #PWR023
+U 1 1 5C002009
+P 5700 4250
+F 0 "#PWR023" H 5700 4100 50  0001 C CNN
+F 1 "+3V3" H 5715 4423 50  0000 C CNN
+F 2 "" H 5700 4250 50  0000 C CNN
+F 3 "" H 5700 4250 50  0000 C CNN
+	1    5700 4250
+	1    0    0    -1
+$EndComp
+$Comp
+L power-supply:+3V3 #PWR014
+U 1 1 5C0020AA
+P 3450 5150
+F 0 "#PWR014" H 3450 5000 50  0001 C CNN
+F 1 "+3V3" H 3465 5323 50  0000 C CNN
+F 2 "" H 3450 5150 50  0000 C CNN
+F 3 "" H 3450 5150 50  0000 C CNN
+	1    3450 5150
+	1    0    0    -1
+$EndComp
+Wire Wire Line
+	10700 1200 10700 1250
+Connection ~ 10700 1200
+Wire Wire Line
+	9850 1200 9850 1150
+Wire Wire Line
+	6350 1500 5750 1500
+Text Label 5850 1500 0    60   ~ 0
+TRANSMIT
+$Comp
+L power-supply:+3V3 #PWR047
+U 1 1 5C0C3B73
+P 6600 3400
+F 0 "#PWR047" H 6600 3250 50  0001 C CNN
+F 1 "+3V3" H 6615 3573 50  0000 C CNN
+F 2 "" H 6600 3400 50  0000 C CNN
+F 3 "" H 6600 3400 50  0000 C CNN
+	1    6600 3400
+	1    0    0    -1
+$EndComp
+$Comp
+L devices:R_0603 R21
+U 1 1 5C0C3F98
+P 2100 7000
+F 0 "R21" H 2130 7020 50  0000 L CNN
+F 1 "4k7" H 2130 6960 50  0000 L CNN
+F 2 "resistors:R_0603" H 2100 6850 50  0001 C CNN
+F 3 "" H 2100 7000 50  0000 C CNN
+	1    2100 7000
+	1    0    0    -1
+$EndComp
+$Comp
+L power-supply:VCC #PWR01
+U 1 1 5C0C40E2
+P 2100 6850
+F 0 "#PWR01" H 2100 6700 50  0001 C CNN
+F 1 "VCC" H 2100 7000 50  0000 C CNN
+F 2 "" H 2100 6850 50  0000 C CNN
+F 3 "" H 2100 6850 50  0000 C CNN
+	1    2100 6850
+	1    0    0    -1
+$EndComp
+Wire Wire Line
+	1750 7250 2100 7250
+Wire Wire Line
+	2100 7250 2100 7100
+Wire Wire Line
+	2100 7100 2400 7100
+Connection ~ 2100 7100
+Wire Wire Line
+	2100 6850 2100 6900
+Wire Wire Line
+	8150 1150 8150 1200
+Wire Wire Line
+	8550 750  8150 750
+Wire Wire Line
+	6200 950  7000 950
+$Comp
+L power-supply:GND #PWR052
+U 1 1 5C1502A8
+P 7750 1200
+F 0 "#PWR052" H 7750 950 50  0001 C CNN
+F 1 "GND" H 7750 1050 50  0000 C CNN
+F 2 "" H 7750 1200 50  0000 C CNN
+F 3 "" H 7750 1200 50  0000 C CNN
+	1    7750 1200
+	1    0    0    -1
+$EndComp
+Wire Wire Line
+	7100 1200 7000 1200
+Wire Wire Line
+	7000 1200 7000 950
+Connection ~ 7000 950
+Wire Wire Line
+	7000 950  7850 950
+Wire Wire Line
+	7300 1200 7450 1200
+Wire Wire Line
+	7650 1200 7750 1200
 $EndSCHEMATC

Commit message: generated production files, pdf and gerber
Other:
- note added: "Copyright generationmake 2018\nsee full project documentation at http://ardutrx.generationmake.de"
- note added: "You may redistribute and modify this documentation under the terms of the CERN OHL v.1.2. (http://ohwr.org/cernohl).\nThis documentation is distributed WITHOUT ANY EXPRESS OR IMPLIED WARRANTY, INCLUDING OF MERCHANTABILITY, SATISFACTORY\nQUALITY AND FITNESS FOR A PARTICULAR PURPOSE. Please see the CERN OHL v.1.2 for applicable conditions"
- note added: "filter according to DMR818 datasheet"
- note added: "place R30 only if no filter necessary"
- note removed: "Copyright generationmake 2018\nsee full project documentation at http://ardutrx.generationmake.de\n\nThis documentation describes Open Hardware and is licensed \nunder the CERN OHL v. 1.2.\nYou may redistribute and modify this documentation under the terms \nof the CERN OHL v.1.2. (http://ohwr.org/cernohl). This documentation \nis distributed WITHOUT ANY EXPRESS OR IMPLIED WARRANTY, \nINCLUDING O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"
- note removed: "filter for 2m version\nchebyshev low pass filter\ncutoff frequency: 185 MHz\npassband ripple: 0.5 dB\nimpedance: 50 Ohm"
- note removed: "place R28..30 only if no filter necessary"
Changed lines of the file:
@@
 encoding utf-8
 Sheet 1 1
-Title "ArduTrx Shield"
-Date "2018-08-21"
-Rev "x1.1"
-Comp ""
+Title "ArduTrxDMR Shield"
+Date "2018-11-27"
+Rev "x1.0"
+Comp "generationmake"
 Comment1 ""
 Comment2 ""
 Comment3 ""
-Comment4 ""
+Comment4 "This documentation describes Open Hardware and is licensed under the CERN OHL v. 1.2."
 $EndDescr
 $Comp
@@
 Text Notes 2550 7600 0    60   ~ 0
 LM4861 also works
-Text Notes 700  3000 0    60   ~ 0
-filter for 2m version\nchebyshev low pass filter\ncutoff frequency: 185 MHz\npassband ripple: 0.5 dB\nimpedance: 50 Ohm
+Text Notes 2500 2750 0    60   ~ 0
+filter according to DMR818 datasheet
 $Comp
 L voltage-regulators:LT1085 U2
@@
 ANT3
 Text Notes 2400 2650 0    60   ~ 0
-place R28..30 only if no filter necessary
+place R30 only if no filter necessary
 Text Notes 500  1350 0    47   ~ 0
-Copyright generationmake 2018\nsee full project documentation at http://ardutrx.generationmake.de\n\nThis   documentation   describes   Open   Hardware   and   is   licensed   \nunder   the CERN OHL v. 1.2.\nYou may redistribute and modify this documentation under the terms \nof the CERN OHL v.1.2. (http://ohwr.org/cernohl). This documentation \nis distributed WITHOUT   ANY   EXPRESS   OR   IMPLIED   WARRANTY, \nINCLUDING   OF MERCHANTABILITY,   SATISFACTORY   QUALITY   AND \nFITNESS   FOR   A PARTICULAR   PURPOSE.   Please   see   the   CERN   \nOHL   v.1.2  for   applicable conditions
+Copyright generationmake 2018\nsee full project documentation at http://ardutrx.generationmake.de
 $Comp
 L devices:CP_Small C15
@@
 Wire Wire Line
 	7650 1200 7750 1200
+Text Notes 7000 6900 0    43   ~ 0
+You may redistribute and modify this documentation under the terms of the CERN OHL v.1.2. (http://ohwr.org/cernohl).\nThis documentation is distributed WITHOUT ANY EXPRESS OR IMPLIED WARRANTY, INCLUDING OF MERCHANTABILITY, SATISFACTORY\nQUALITY AND FITNESS FOR A PARTICULAR PURPOSE. Please see the CERN OHL v.1.2 for applicable conditions
 $EndSCHEMATC
