File: hardware/DummyLoad/kicad_source/DummyLoad/DummyLoad.kicad_pcb (KiCad board)
At the start: 2 copper layers, 34 x 40 mm, 55 parts, among them CN1 60312202114509, CN2 60312202114509

Commit message: added comments to schematic, added laber with license to pcb
Parts:
- CN1, CN2: value 60312202114509 -> CON-SMA-EDGE-S-ND
Other:
- board text added: "Licensed under CERN OHL v 1.2"
Changed lines of the file:
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@@
   (general
     (thickness 1.6)
-    (drawings 19)
+    (drawings 20)
     (tracks 197)
     (zones 0)
@@
   )
   (setup
-    (last_trace_width 1.3)
+    (last_trace_width 0.25)
     (user_trace_width 1.3)
     (trace_clearance 0.2)
@@
       (effects (font (size 1 1) (thickness 0.15)))
     )
-    (fp_text value 60312202114509 (at 0 -0.5 180) (layer F.Fab)
+    (fp_text value CON-SMA-EDGE-S-ND (at 0 -0.5 180) (layer F.Fab)
       (effects (font (size 1 1) (thickness 0.15)))
     )
@@
       (effects (font (size 1 1) (thickness 0.15)))
     )
-    (fp_text value 60312202114509 (at 0 -0.5) (layer F.Fab)
+    (fp_text value CON-SMA-EDGE-S-ND (at 0 -0.5) (layer F.Fab)
       (effects (font (size 1 1) (thickness 0.15)))
     )
@@
       (xy 5.541591 2.802653)) (layer B.SilkS) (width 0.01))
   )
+  (gr_text "Licensed under \nCERN OHL v 1.2" (at 87.5 113.5 90) (layer B.SilkS)
+    (effects (font (size 1 1) (thickness 0.25)) (justify mirror))
+  )
   (gr_circle (center 87 104) (end 89 104) (layer B.Mask) (width 2))
