File: kicad_source/ArduTrxShield.kicad_pcb (KiCad board)
At the start: 2 copper layers, 84.8 x 53 mm, 81 parts, among them CN1 60312202114509, CN2 ARDUINO, CN3 CON_KLINKE3, CN4 CON_KLINKE3, CN5 CONN_01X03, CN6 CONN_01X02, CN7 691322310002, Q1 2N7002, Q2 2N7002, Q3 2N7002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

Commit message: updated bom, added part numbers
Parts:
- C1, C4: value 30p -> 30pF
- C10, C11, C12, C14, C16, C17, C18, C19, C20, C5, C7, C8: value 100n -> 100nF
- C15: value 470u -> 470uF
- C2, C3: value 47p -> 47pF
- C6, C9: value 10u -> 10uF
- CN5: value CONN_01X03 -> 61300311121
- CN6: value CONN_01X02 -> 61300211121
- D1: value Led_red -> 150060RS75000
- D2: value Led_yellow -> 150060YS75000
- D3: value Led_green -> 150060GS75000
- S1: value SW_DIP_x1 -> 418117270901
- SW1: value TAST_HOR -> 431256058736
- SW2: value ALPS_EC11E -> 482009514001
- U2: value LT1085 -> LM1085IS-ADJ

Commit message: updated part numbers
Parts:
- C13: value 1u -> 1uF
- C15: value 470uF -> UWT1A471MNL1GS
- CN3: value CON_KLINKE3 -> LUM 1503-07
- CN4: value CON_KLINKE3 -> LUM 1501-03
Changed lines of the file:
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@@
       (effects (font (size 1 1) (thickness 0.15)))
     )
-    (fp_text value CON_KLINKE3 (at 0 6) (layer F.Fab)
+    (fp_text value "LUM 1501-03" (at 0 6) (layer F.Fab)
       (effects (font (size 1 1) (thickness 0.15)))
     )
@@
       (effects (font (size 1 1) (thickness 0.15)))
     )
-    (fp_text value 470uF (at 0 5.08 180) (layer F.Fab)
+    (fp_text value UWT1A471MNL1GS (at 0 5.08 180) (layer F.Fab)
       (effects (font (size 1 1) (thickness 0.15)))
     )
@@
       (effects (font (size 1 1) (thickness 0.15)))
     )
-    (fp_text value 1u (at 0 1.9 180) (layer F.Fab)
+    (fp_text value 1uF (at 0 1.9 180) (layer F.Fab)
       (effects (font (size 1 1) (thickness 0.15)))
     )
@@
       (effects (font (size 1 1) (thickness 0.15)))
     )
-    (fp_text value CON_KLINKE3 (at 0 6) (layer F.Fab)
-      (effects (font (size 1 1) (thickness 0.15)))
-    )
+    (fp_text value "LUM 1503-07" (at 0 6) (layer F.Fab)
+      (effects (font (size 1 1) (thickness 0.15)))
+    )
