File: kicad_source/ArduTrxShield.sch (KiCad schematic (older format))
At the start: 81 parts, among them CN1 60312202114509, CN2 ARDUINO, CN3 CON_KLINKE3, CN4 CON_KLINKE3, CN5 CONN_01X03, CN6 CONN_01X02, CN7 691322310002, Q1 2N7002, Q2 2N7002, Q3 2N7002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

Commit message: updated to latest kicad version
Parts:
- CN2: symbol MODULE_compute:ARDUINO -> ArduTrxShield-rescue:ARDUINO-MODULE_compute
Other:
- moved on the sheet: CN2
Changed lines of the file:
@@
 EESchema Schematic File Version 4
-LIBS:ATX_connector
-LIBS:CAN-transceiver
-LIBS:come_connector
-LIBS:CON_wuerth
-LIBS:D_esdprotection
-LIBS:devices
-LIBS:displayport_connector
-LIBS:displays
-LIBS:electrical-connectors
-LIBS:eth_usb_connectors_combos
-LIBS:ftdi
-LIBS:IC_batterycharger
-LIBS:IC_clockbuffer
-LIBS:IC_interface_i2c
-LIBS:IC_levelshifter
-LIBS:IC_loadswitch
-LIBS:IC_microcontroller_ST
-LIBS:IC_rtc
-LIBS:IC_sensor
-LIBS:IC_transceiver_can
-LIBS:IC_transceiver_rs
-LIBS:IC_usbhub
-LIBS:interface
-LIBS:LED-controllers
-LIBS:L_filter
-LIBS:L_power
-LIBS:mechanical-connectors
-LIBS:mechanical-switches
-LIBS:MECH_smd-contact-finger
-LIBS:MECH_smd-mounting
-LIBS:MECH_smd-spacer
-LIBS:MEMS
-LIBS:microcontrollers
-LIBS:MODULE_compute
-LIBS:motor-driver
-LIBS:opamps
-LIBS:PCB_touch
-LIBS:PCIe_connectors
-LIBS:power-monitors
-LIBS:power-supply
-LIBS:sata_con
-LIBS:transistors
-LIBS:usb_connector_header
-LIBS:voltage-regulators
-LIBS:MODULE_RF
-LIBS:IC_audio
-LIBS:ArduTrxShield-cache
-EELAYER 26 0
+EELAYER 30 0
 EELAYER END
 $Descr A4 11693 8268
@@
 $EndDescr
 $Comp
-L MODULE_compute:ARDUINO CN2
+L ArduTrxShield-rescue:ARDUINO-MODULE_compute CN2
 U 1 1 5B0B2CBD
 P 10100 3250

Commit message: updated bom, added part numbers
Parts:
- C1, C4: value 30p -> 30pF
- C10, C11, C12, C14, C16, C17, C18, C19, C20, C5, C7, C8: value 100n -> 100nF
- C13: value 1u -> 1uF
- C15: value 470u -> 470uF
- C2, C3: value 47p -> 47pF
- C6, C9: value 10u -> 10uF
- CN5: value CONN_01X03 -> 61300311121
- CN6: value CONN_01X02 -> 61300211121
- D1: value Led_red -> 150060RS75000
- D2: value Led_yellow -> 150060YS75000
- D3: value Led_green -> 150060GS75000
- S1: value SW_DIP_x1 -> 418117270901
- SW1: value TAST_HOR -> 431256058736
- SW2: value ALPS_EC11E -> 482009514001
- U2: value LT1085 -> LM1085IS-ADJ
Changed lines of the file:
@@
 Sheet 1 1
 Title "ArduTrx Shield"
-Date "2018-08-21"
-Rev "x1.1"
-Comp ""
+Date "2020-11-29"
+Rev "x1.1.1"
+Comp "generationmake"
 Comment1 ""
 Comment2 ""
@@
 P 6200 1150
 F 0 "D3" H 6150 1275 50  0000 L CNN
-F 1 "Led_green" H 6025 1050 50  0000 L CNN
+F 1 "150060GS75000" H 6025 1050 50  0000 L CNN
 F 2 "LEDs:LED_0603" V 6200 1150 50  0001 C CNN
 F 3 "" V 6200 1150 50  0000 C CNN
@@
 P 5800 3450
 F 0 "C5" H 5810 3520 50  0000 L CNN
-F 1 "100n" H 5810 3370 50  0000 L CNN
+F 1 "100nF" H 5810 3370 50  0000 L CNN
 F 2 "capacitors:C_0603" H 5800 3300 50  0001 C CNN
 F 3 "" H 5800 3450 50  0000 C CNN
@@
 P 8400 5150
 F 0 "CN5" H 8400 5350 50  0000 C CNN
-F 1 "CONN_01X03" V 8500 5150 50  0000 C CNN
+F 1 "61300311121" V 8500 5150 50  0000 C CNN
 F 2 "pin_headers:Pin_Header_Straight_1x03" H 8400 5150 50  0001 C CNN
 F 3 "" H 8400 5150 50  0000 C CNN
@@
 P 10500 1200
 F 0 "D2" H 10450 1325 50  0000 L CNN
-F 1 "Led_yellow" H 10325 1100 50  0000 L CNN
+F 1 "150060YS75000" H 10325 1100 50  0000 L CNN
 F 2 "LEDs:LED_0603" V 10500 1200 50  0001 C CNN
 F 3 "" V 10500 1200 50  0000 C CNN
@@
 P 10500 800
 F 0 "D1" H 10450 925 50  0000 L CNN
-F 1 "Led_red" H 10325 700 50  0000 L CNN
+F 1 "150060RS75000" H 10325 700 50  0000 L CNN
 F 2 "LEDs:LED_0603" V 10500 800 50  0001 C CNN
 F 3 "" V 10500 800 50  0000 C CNN
@@
 P 4250 2150
 F 0 "C4" H 4260 2220 50  0000 L CNN
-F 1 "30p" H 4260 2070 50  0000 L CNN
+F 1 "30pF" H 4260 2070 50  0000 L CNN
 F 2 "capacitors:C_0603" H 4250 2000 50  0001 C CNN
 F 3 "" H 4250 2150 50  0000 C CNN
@@
 P 3650 2150
 F 0 "C3" H 3660 2220 50  0000 L CNN
-F 1 "47p" H 3660 2070 50  0000 L CNN
+F 1 "47pF" H 3660 2070 50  0000 L CNN
 F 2 "capacitors:C_0603" H 3650 2000 50  0001 C CNN
 F 3 "" H 3650 2150 50  0000 C CNN
@@
 P 3050 2150
 F 0 "C2" H 3060 2220 50  0000 L CNN
-F 1 "47p" H 3060 2070 50  0000 L CNN
+F 1 "47pF" H 3060 2070 50  0000 L CNN
 F 2 "capacitors:C_0603" H 3050 2000 50  0001 C CNN
 F 3 "" H 3050 2150 50  0000 C CNN
@@
 P 2450 2150
 F 0 "C1" H 2460 2220 50  0000 L CNN
-F 1 "30p" H 2460 2070 50  0000 L CNN
+F 1 "30pF" H 2460 2070 50  0000 L CNN
 F 2 "capacitors:C_0603" H 2450 2000 50  0001 C CNN
 F 3 "" H 2450 2150 50  0000 C CNN
@@
 P 1450 6500
 F 0 "C10" H 1460 6570 50  0000 L CNN
-F 1 "100n" H 1460 6420 50  0000 L CNN
+F 1 "100nF" H 1460 6420 50  0000 L CNN
 F 2 "capacitors:C_0603" H 1450 6350 50  0001 C CNN
 F 3 "" H 1450 6500 50  0000 C CNN
@@
 P 2300 7300
 F 0 "C13" H 2310 7370 50  0000 L CNN
-F 1 "1u" H 2310 7220 50  0000 L CNN
+F 1 "1uF" H 2310 7220 50  0000 L CNN
 F 2 "capacitors:C_0603" H 2300 7150 50  0001 C CNN
 F 3 "" H 2300 7300 50  0000 C CNN
@@
 P 3550 6750
 F 0 "C11" H 3560 6820 50  0000 L CNN
-F 1 "100n" H 3560 6670 50  0000 L CNN
+F 1 "100nF" H 3560 6670 50  0000 L CNN
 F 2 "capacitors:C_0603" H 3550 6600 50  0001 C CNN
 F 3 "" H 3550 6750 50  0000 C CNN
@@
 P 3950 7150
 F 0 "C12" H 3960 7220 50  0000 L CNN
-F 1 "100n" H 3960 7070 50  0000 L CNN
+F 1 "100nF" H 3960 7070 50  0000 L CNN
 F 2 "capacitors:C_0603" H 3950 7000 50  0001 C CNN
 F 3 "" H 3950 7150 50  0000 C CNN
@@
 P 4700 6950
 F 0 "CN6" H 4700 7100 50  0000 C CNN
-F 1 "CONN_01X02" V 4800 6950 50  0000 C CNN
+F 1 "61300211121" V 4800 6950 50  0000 C CNN
 F 2 "pin_headers:Pin_Header_Straight_1x02" H 4700 6950 50  0001 C CNN
 F 3 "" H 4700 6950 50  0000 C CNN
@@
 P 3150 3700
 F 0 "U2" H 2750 3950 60  0000 C CNN
-F 1 "LT1085" H 2850 3500 60  0000 C CNN
+F 1 "LM1085IS-ADJ" H 2850 3500 60  0000 C CNN
 F 2 "SOT_TO:TO-263-3Lead" H 3100 3400 60  0001 C CNN
 F 3 "" H 3150 3700 60  0000 C CNN
@@
 P 4450 3750
 F 0 "C8" H 4460 3820 50  0000 L CNN
-F 1 "100n" H 4460 3670 50  0000 L CNN
+F 1 "100nF" H 4460 3670 50  0000 L CNN
 F 2 "capacitors:C_0603" H 4450 3600 50  0001 C CNN
 F 3 "" H 4450 3750 50  0000 C CNN
@@
 P 4800 3750
 F 0 "C9" H 4810 3820 50  0000 L CNN
-F 1 "10u" H 4810 3670 50  0000 L CNN
+F 1 "10uF" H 4810 3670 50  0000 L CNN
 F 2 "capacitors:C_0805" H 4800 3600 50  0001 C CNN
 F 3 "" H 4800 3750 50  0000 C CNN
@@
 P 2000 3750
 F 0 "C7" H 2010 3820 50  0000 L CNN
-F 1 "100n" H 2010 3670 50  0000 L CNN
+F 1 "100nF" H 2010 3670 50  0000 L CNN
 F 2 "capacitors:C_0603" H 2000 3600 50  0001 C CNN
 F 3 "" H 2000 3750 50  0000 C CNN
@@
 P 1600 3750
 F 0 "C6" H 1610 3820 50  0000 L CNN
-F 1 "10u" H 1610 3670 50  0000 L CNN
+F 1 "10uF" H 1610 3670 50  0000 L CNN
 F 2 "capacitors:C_0805" H 1600 3600 50  0001 C CNN
 F 3 "" H 1600 3750 50  0000 C CNN
@@
 P 8200 6350
 F 0 "SW2" H 8750 7050 60  0000 C CNN
-F 1 "ALPS_EC11E" H 8750 6300 60  0000 C CNN
+F 1 "482009514001" H 8750 6300 60  0000 C CNN
 F 2 "mechanical-switches:ALPS_EC11E" H 9050 6400 60  0001 C CNN
 F 3 "" H 9050 6400 60  0000 C CNN
@@
 P 3250 5450
 F 0 "C14" H 3260 5520 50  0000 L CNN
-F 1 "100n" H 3260 5370 50  0000 L CNN
+F 1 "100nF" H 3260 5370 50  0000 L CNN
 F 2 "capacitors:C_0603" H 3250 5300 50  0001 C CNN
 F 3 "" H 3250 5450 50  0000 C CNN
@@
 P 7300 2550
 F 0 "SW1" H 7300 2750 60  0000 C CNN
-F 1 "TAST_HOR" H 7300 2350 60  0000 C CNN
+F 1 "431256058736" H 7300 2350 60  0000 C CNN
 F 2 "mechanical-switches:WE_4312x6xxx7x6" H 8150 2600 60  0001 C CNN
 F 3 "" H 8150 2600 60  0000 C CNN
@@
 P 3950 6050
 F 0 "C15" H 3960 6120 50  0000 L CNN
-F 1 "470u" H 3960 5970 50  0000 L CNN
+F 1 "470uF" H 3960 5970 50  0000 L CNN
 F 2 "capacitors:c_elec_8x10.5" H 3950 6050 50  0001 C CNN
 F 3 "" H 3950 6050 50  0000 C CNN
@@
 P 6300 4400
 F 0 "C20" H 6310 4470 50  0000 L CNN
-F 1 "100n" H 6310 4320 50  0000 L CNN
+F 1 "100nF" H 6310 4320 50  0000 L CNN
 F 2 "capacitors:C_0603" H 6300 4250 50  0001 C CNN
 F 3 "" H 6300 4400 50  0000 C CNN
@@
 P 6000 4400
 F 0 "C19" H 6010 4470 50  0000 L CNN
-F 1 "100n" H 6010 4320 50  0000 L CNN
+F 1 "100nF" H 6010 4320 50  0000 L CNN
 F 2 "capacitors:C_0603" H 6000 4250 50  0001 C CNN
 F 3 "" H 6000 4400 50  0000 C CNN
@@
 P 5700 4400
 F 0 "C18" H 5710 4470 50  0000 L CNN
-F 1 "100n" H 5710 4320 50  0000 L CNN
+F 1 "100nF" H 5710 4320 50  0000 L CNN
 F 2 "capacitors:C_0603" H 5700 4250 50  0001 C CNN
 F 3 "" H 5700 4400 50  0000 C CNN
@@
 P 5400 4400
 F 0 "C17" H 5410 4470 50  0000 L CNN
-F 1 "100n" H 5410 4320 50  0000 L CNN
+F 1 "100nF" H 5410 4320 50  0000 L CNN
 F 2 "capacitors:C_0603" H 5400 4250 50  0001 C CNN
 F 3 "" H 5400 4400 50  0000 C CNN
@@
 P 5950 3600
 F 0 "C16" H 5960 3670 50  0000 L CNN
-F 1 "100n" H 5960 3520 50  0000 L CNN
+F 1 "100nF" H 5960 3520 50  0000 L CNN
 F 2 "capacitors:C_0603" H 5950 3450 50  0001 C CNN
 F 3 "" H 5950 3600 50  0000 C CNN
@@
 P 8700 3500
 F 0 "S1" H 8700 3400 50  0000 C CNN
-F 1 "SW_DIP_x1" H 8700 3600 50  0000 C CNN
+F 1 "418117270901" H 8700 3600 50  0000 C CNN
 F 2 "mechanical-switches:dip_1-300" H 8650 3500 50  0001 C CNN
 F 3 "" H 8650 3500 50  0000 C CNN

Commit message: updated part numbers
Parts:
- removed CN2: ARDUINO, MODULE_compute:ARDUINO, symbol ArduTrxShield-rescue:ARDUINO-MODULE_compute
- added CN2: ARDUINO, MODULE_compute:ARDUINO, symbol MODULE_compute:ARDUINO
- C15: value 470uF -> UWT1A471MNL1GS
- CN3: value CON_KLINKE3 -> LUM 1503-07
- CN4: value CON_KLINKE3 -> LUM 1501-03
Other:
- note added: "470 uF"
Changed lines of the file:
@@
 $EndDescr
-$Comp
-L ArduTrxShield-rescue:ARDUINO-MODULE_compute CN2
-U 1 1 5B0B2CBD
-P 10100 3250
-F 0 "CN2" H 10200 5000 60  0000 C CNN
-F 1 "ARDUINO" H 10300 1400 60  0000 C CNN
-F 2 "MODULE_compute:ARDUINO" H 10650 5000 60  0001 C CNN
-F 3 "" H 10750 4050 60  0000 C CNN
-	1    10100 3250
-	1    0    0    -1
-$EndComp
 $Comp
 L MODULE_RF:DRA818 U1
@@
 P 5150 6050
 F 0 "CN4" H 5100 6250 60  0000 C CNN
-F 1 "CON_KLINKE3" H 5100 5900 60  0000 C CNN
+F 1 "LUM 1501-03" H 5100 5900 60  0000 C CNN
 F 2 "CON_lumberg:1501_03" H 5150 6050 60  0001 C CNN
 F 3 "" H 5150 6050 60  0000 C CNN
@@
 P 5150 5250
 F 0 "CN3" H 5100 5450 60  0000 C CNN
-F 1 "CON_KLINKE3" H 5100 5100 60  0000 C CNN
+F 1 "LUM 1503-07" H 5100 5100 60  0000 C CNN
 F 2 "CON_lumberg:1503_07" H 5150 5250 60  0001 C CNN
 F 3 "" H 5150 5250 60  0000 C CNN
@@
 P 3950 6050
 F 0 "C15" H 3960 6120 50  0000 L CNN
-F 1 "470uF" H 3960 5970 50  0000 L CNN
+F 1 "UWT1A471MNL1GS" H 3960 5970 50  0000 L CNN
 F 2 "capacitors:c_elec_8x10.5" H 3950 6050 50  0001 C CNN
 F 3 "" H 3950 6050 50  0000 C CNN
@@
 Wire Wire Line
 	8250 2500 8400 2500
+Text Notes 3450 6100 0    60   ~ 0
+470 uF
+$Comp
+L MODULE_compute:ARDUINO CN2
+U 1 1 5FE53E6E
+P 10100 3250
+F 0 "CN2" H 10719 3258 60  0000 L CNN
+F 1 "ARDUINO" H 10719 3152 60  0000 L CNN
+F 2 "MODULE_compute:ARDUINO" H 10650 5000 60  0001 C CNN
+F 3 "" H 10750 4050 60  0000 C CNN
+	1    10100 3250
+	1    0    0    -1
+$EndComp
 $EndSCHEMATC
